Commit message: fixed nao urdf

File: src/RelaxedIK/urdfs/nao_v4.urdf (robot description, URDF)
Before this commit: robot NaoH25V40, 83 links, 82 joints
Joints:
- joint LHipYawPitch: axis 0 0.707106 -0.707106 -> 1 0 0
- joint RHipYawPitch: axis 0 0.707106 0.707106 -> 1 0 0

Commit message: added fixed joints to end effectors of arms, prep for direct control joints

File: src/RelaxedIK/urdfs/nao_v4.urdf (robot description, URDF)
Before this commit: robot NaoH25V40, 83 links, 82 joints
Links:
- added link l_palm
- added link r_palm
Joints:
- added joint LArm_effector_fixedjoint: type fixed, parent l_wrist, child l_palm, origin xyz=0 0 0 rpy=0 0 0, axis -0.4017 -0.2659 -0.1617
- added joint RArm_effector_fixedjoint: type fixed, parent r_wrist, child r_palm, origin xyz=0 0 0 rpy=0 0 0, axis 0.4017 -0.2659 0.1617
