Commit message: bug fixes and switches for wiscutils

File: src/RelaxedIK/urdfs/pepper_modified.urdf (robot description, URDF)
Before this commit: robot JulietteY20MP, 86 links, 85 joints
Joints:
- joint LArm_effector_fixedjoint: axis 1.0 0 0 -> 0 0 0; limit lower=0.02 upper=0.98 effort=0.144 velocity=12.56 -> (none); origin xyz=0.025 0 0 rpy=0 0 0 -> xyz=0 0 0 rpy=0 0 0
- joint RArm_effector_fixedjoint: axis 1.0 0 0 -> 0 0 0; limit lower=0.02 upper=0.98 effort=0.144 velocity=12.56 -> (none); origin xyz=0.025 0 0 rpy=0 0 0 -> xyz=0 0 0 rpy=0 0 0
