Commit message: misc

File: config/urdfs/fetch.urdf (robot description, URDF)
Before this commit: robot fetch, 26 links, 25 joints
Links:
- link estop_link: geometry collision mesh filename=package://fetch_description/meshes/estop_link.STL; visual mesh filename=package://fetch_description/meshes/estop_link.dae
Joints:
- joint forearm_roll_joint: limit effort=29.35 velocity=1.571 -> lower=-15. upper=15.0 effort=29.35 velocity=1.571
- joint upperarm_roll_joint: limit effort=76.94 velocity=1.571 -> lower=-15. upper=15.0 effort=76.94 velocity=1.571
- joint wrist_roll_joint: limit effort=7.36 velocity=2.268 -> lower=-15. upper=15.0 effort=7.36 velocity=2.268
